File: zulu_a7.sch (EAGLE design)
At the start: 177 parts, among them J1 Pmod 2x6, Q1 12MHz 25ppm (FPGA + FT2232HQ), Q2 NMOS, Q3 MBT3904DW1T1, U1 XC7A35T-1CPG236C, U10 93LC46BT-I/SN, U2 FT2232HQ USB-UART/JTAG Bridge, U3 AS4C32M16SB-6TIN, U4 W25Q128JVSIQ, U8 LTC3569EUDC#TRPBF, X1 Molex 105017-0001 Micro-USB-B, X2 ZULU-CONN, X3 MICROSD_CONDM3AT-SF-PEJM5

Commit message: The 22 HF decoupling caps go 0402 -> 0201, and the board is fully placed
Option A: package only, value untouched. New C0201 package in rcl on the same
land as R0201 -- C0402 and R0402 already share theirs, so the pair follows -- and
a C0201 device on C-US.

IT PUT THEM CLOSER, WHICH IS THE POINT. Distance from the ball centre goes
min 8.4 -> 5.1, median 9.3 -> 6.8, max 9.7 -> 10.9. The median moving 2.5 mm in
is worth more than the one outlier moving out: a bypass capacitor's loop is what
it costs you, and a smaller body reaches nearer the ball it serves. Lower ESL on
top of that is why Cmod A7 does it.

WHAT IT COSTS, RECORDED ON ALL 22 AS A NOTE RATHER THAN LEFT TO BE REDISCOVERED.
The 16 V GRM155R61C474KA88D becomes a 6.3 V 0201. On VCC3V3 that part sits at
52 % of rating, where DC bias typically takes 60-75 % of the capacitance against
15-25 % for the 16 V 0402. The BOM value does not change, so validate.py's UG483
count still reads 16/8/2 and passes -- it counts nominal values and cannot see
bias derating. Effective decoupling on the 3V3 rail is roughly half what it was.
That is the trade the ESL and the placement bought, and it should be checked
against Murata's bias curves before this is ordered, along with the MPN suffix.

The 4.7 uF and the 47 uF stay where they are. Not a judgement -- 0201 tops out
around 1 to 2.2 uF, so there is no part to convert them to.

C124 is untouched. It is the same GRM155R61C474KA88D and would have been swept
up by a global replace, but it is a 470 nF on FPGA CONNECT, not U1 decoupling on
sheet 7. An assertion on the MPN count caught it: 23 in the file, 22 on the sheet.

Every real part is now on the board. 172 placed, 0 parked -- the only things
below the outline are the four padless CC artwork blocks, which are parked by
design. check_board and validate 0 findings.

Co-Authored-By: Claude Opus 5 <noreply@anthropic.com>
Parts:
- C107, C108, C109, C110, C111, C112, C113, C114, C115, C116, C117, C118, C119, C120, C121, C122, C89, C90, C91, C92, C95, C96: device rcl:C-USC0402 -> rcl:C-USC0201; MANF# GRM155R61C474KA88D -> GRM033R60J474KE15D; NOTE (none) -> 0402 -> 0201 to cut ESL, following Cmod A7. THE VOLTAGE RAT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; SPEC X5R 16V +-10%, 0.50 mm max -> X5R 6.3V +-10%, 0.30 mm max

Commit message: No 1206 left: the bulk becomes twelve 22uF 0805
Each 47uF 1206 splits in two. Nominal per position falls 47 -> 44 uF, but the
0805 is 10 V where the 1206 was 6.3 V, so it derates less under bias and the
pair should deliver at least what the single part did. Height drops 1.60 -> 1.45
mm, which the back-side budget against the 2.54 mm header standoff cares about.
Totals: VCC1V0 6, VCC1V8 2, VCC3V3 4.

The six siblings needed somewhere to be drawn, and every ladder on sheet 7 was
full -- one free slot at x 60.96, and two of the rows reach their rail through a
supply symbol rather than a labelled run. So three new rows go in the empty band
at y 98..151, x 5..30, each with its own rail, GND rail and GND supply
(GND40-42). New segments inside the existing net elements, so they are the same
net by construction and no existing wire moved.

validate.py's UG483 table is updated with them -- it hardcodes counts per rail,
so this was not bookkeeping: 47uF/3/1/2 becomes 22uF/6/2/4.

TWO THINGS THIS TAUGHT ME, BOTH RECORDED WHERE THEY BIT.

Junctions. The rule is cnt + 2*through + (1 if a pin is there) >= 3, so a GND
supply pin with a stub and a rail meeting at it needs a junction even though
only two wires end there. Two were missing and validate named the coordinates.

X3 carries a 0.15 mm CIRCLE on layer 21 at local (4.6, 1.1), and the socket is
rotated R270, which swings that circle out to x 17.20 -- past every wire in the
package. My free-space map read wires and rectangles and not circles, so it
offered C98 a slot at 16.65 that the generator then rejected. The map now reads
circles too.

Two 0805 want more board than one 1206 once each carries its own keepout and
gap, so doubling the count cost area even though every part got smaller: three
of the twelve had no seat, then a fourth fell out when I pinned them. C86, C93,
C97 and C98 are pinned by hand at the REGULATOR, 12.5 to 14.4 mm from U8, which
is where this file already says bulk belongs -- it gains nothing from sitting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
Parts:
- added C141, C142, C143, C144, C145, C146: 22uF, rcl:C-USC0805
- C140, C85, C86, C93, C97, C98: value 47uF -> 22uF; device rcl:C-USC1206 -> rcl:C-USC0805; MANF# GRM31CR60J476ME19L -> GRM21BR61A226ME44L; SPEC X5R 6.3V +-20%, 1.60 mm MAX -- back side, see board/STACKUP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 -> X5R 10V +-20%, 1.45 mm max
Connections:
- net GND: now also C141.2, C142.2, C143.2, C144.2, C145.2, C146.2
- net VCC1V0: now also C141.1, C142.1, C143.1
- net VCC1V8: now also C144.1
- net VCC3V3: now also C145.1, C146.1

Commit message: U2's support drops to 0201 where the physics allows: 24 of 36
Fifteen resistors and nine capacitors on the FT2232's sheet.

THE RESISTORS ARE NOT CLOSE TO ANY LIMIT. Every one converted is a pull-up,
pull-down or high-value series: the ten 10k at 1.1 mW, R99 at 2.3, R5 at 2.1,
R101 at 4.9, R24/R25 carrying AC only at about 1.3. Against an 0201's 50 mW
that is 2 to 10 percent. R5 was the last 0603 on the sheet and is now 0201 with
it; it also loses a non-Yageo part number for the same series as its siblings.

THE CAPACITORS ARE THE POINT, THOUGH. 0.1 uF is the value where 0201 actually
works -- bias derating at 0.1 uF is mild, which is exactly what it is not at the
0.47 uF on sheet 7. And C40 and C41 sit on FT-VPHY and FT-VPLL, the USB PHY and
PLL supplies, where lower ESL is worth having rather than merely tolerable.

But the dielectric changes and that is recorded on every one: X7R 16V becomes
X5R 10V, because 0201 at this capacitance is an X5R part. X5R stops at +85 C
where X7R goes to +125. Fine for this board, not a like-for-like swap. C38 drops
50V to 25V, which was over-specified for a 3.3V rail either way.

TWO DID NOT MOVE AND BOTH SAY WHY ON THE PART.
  R100  330R holding DONE low through configuration is 33 mW: 53 percent of an
        0402 but 66 of an 0201, sustained for all of config and indefinitely if
        config fails. 330R on DONE is standard Xilinx practice, so the value is
        not the thing to change -- the package is where the margin is.
  R18   the FT2232's RREF, which sets USB transceiver bias. 0.9 mW and 1 percent
        is 1 percent at any size, but there is no space pressure left on this
        board, so there is nothing to win against a part whose drift shows up as
        signal quality.

The six 100R JTAG series stay 0402 for the reason already recorded when R4 was
split, and C39/C139 stay because 3.3 uF does not exist in 0201.

CHECK_BOARD CAUGHT A BUG VALIDATE DID NOT. All nine capacitors are on C-GENERIC,
not C-US, and C-GENER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
Parts:
- C133, C134, C135, C136, C137, C138: device rcl:C-GENERICC0402 -> rcl:C-GENERICC0201; MANF# GRM155R71C104KA88D -> GRM033R61A104KE15D; NOTE (none) -> 0402 -> 0201 on U2's support. The DIELECTRIC AND VOLTAGE BO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; SPEC X7R 16V +-10%, 0.50 mm max -> X5R 10V +-10%, 0.30 mm max
- C38: device rcl:C-GENERICC0402 -> rcl:C-GENERICC0201; MANF# GRM155R71H103KA88D -> GRM033R71E103KE14D; NOTE (none) -> 0402 -> 0201 on U2's support. 50V drops to 25V, which is st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; SPEC X7R 50V +-10%, 0.50 mm max -> X7R 25V +-10%, 0.30 mm max
- C40, C41: device rcl:C-GENERICC0402 -> rcl:C-GENERICC0201; MANF# GRM155R71C104KA88D -> GRM033R61A104KE15D; NOTE (none) -> 0402 -> 0201 on U2's support. The DIELECTRIC AND VOLTAGE BO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; SPEC X7R 16V +-10%, 0.50 mm max -- same part as the 0.1uF line -> X5R 10V +-10%, 0.30 mm max
- R100: NOTE (none) -> Stays 0402 deliberately. At 330R holding DONE low through c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
- R101: device rcl:R-US_SMALLR0402 -> rcl:R-US_SMALLR0201; MANF# RC0402FR-072K21L -> RC0201FR-072K21L; SPEC thick film +-1%, 1/16W, 0402 -> thick film +-1%, 1/20W, 0201
- R18: NOTE (none) -> Stays 0402 deliberately. Power is trivial (0.9 mW) and 1 pe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
- R19, R89, R90, R91, R92, R93, R94, R96, R97, R98: device rcl:R-US_SMALLR0402 -> rcl:R-US_SMALLR0201; MANF# RC0402FR-0710KL -> RC0201FR-0710KL; SPEC thick film +-1%, 1/16W, 0402 -> thick film +-1%, 1/20W, 0201
- R24, R25: device rcl:R-US_SMALLR0402 -> rcl:R-US_SMALLR0201; MANF# RC0402FR-0733RL -> RC0201FR-0733RL; SPEC thick film +-1%, 1/16W, 0402 -> thick film +-1%, 1/20W, 0201
- R5: device rcl:R-US_R0603 -> rcl:R-US_R0201; MANF Xicon -> Yageo; MANF# 301-5.1K-RC -> RC0201FR-075K1L; SPEC (none) -> thick film +-1%, 1/20W, 0201
- R99: device rcl:R-US_SMALLR0402 -> rcl:R-US_SMALLR0201; MANF# RC0402FR-074K7L -> RC0201FR-074K7L; SPEC thick film +-1%, 1/16W, 0402 -> thick film +-1%, 1/20W, 0201

Commit message: LD5 and Q2 get part numbers, chosen from what the circuit needs
Both carried no value and no part number, so neither could be ordered. Neither
was recovered from anywhere -- these are selections, and the reasoning is on the
parts as NOTEs rather than in my head.

Q2 -> 2N7002 (onsemi 2N7002LT1G). It switches the PGOOD indicator. Its gate sits
on PGOOD, the LTC3569's open-drain output pulled to 3V3 through R77's 100k, so
Vgs is a static 3.3 V -- a gate draws no DC, which is why a 100k pull-up is fine
here. That demands a LOGIC-LEVEL threshold, and the 2N7002's 1.0 to 2.5 V is
comfortably under 3.3. Drain carries 1.9 mA against 115, and sees 3.3 V against
60. The SOT23-3 footprint names its pads G, S and D at pins 1, 2 and 3, which is
the 2N7002 pinout exactly, so no layout changes.

LD5 -> green 0603 (Lite-On LTST-C191KGKT). THE RESISTOR HAD ALREADY CHOSEN THE
COLOUR and I only had to read it: R78 is 680R off 3.3 V, so the current is
(3.3 - Vf)/680 -- 1.9 mA green, 2.1 red, but 0.6 mA blue or white, too dim to
read across a room. So it was always a green or red part, and green is what
power-good means. Take R78 to 330R if 1.9 mA is too faint.

A bare "<" is not legal in an XML attribute, and my first SPEC said "Vf <= 2.1V".
The file stopped parsing at that character. Rewritten as "2.1V max"; git had the
good copy.

bom.py now says what a PermissionError means. Excel takes an exclusive lock on an
open csv, and the traceback reads like a filesystem fault while the stale file
sits there looking fresh -- which is exactly how I first read the blank fields
back. docs/zulu_a7-bom.csv is NOT regenerated in this commit for that reason:
close it and re-run tools/bom.py.

Co-Authored-By: Claude Opus 5 <noreply@anthropic.com>
Parts:
- LD5: value (none) -> green; MANF (none) -> Lite-On; MANF# (none) -> LTST-C191KGKT; NOTE (none) -> Power-good indicator: VCC3V3 to LD5 to R78 680R to Q2 drain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; SPEC (none) -> green indicator, 0603, Vf 2.1V max at 2mA
- Q2: value NMOS -> 2N7002; MANF (none) -> onsemi; MANF# (none) -> 2N7002LT1G; NOTE (none) -> Switches the PGOOD indicator LD5. SELECTED FROM THE CIRCUIT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; SPEC (none) -> N-ch MOSFET, logic level: Vgs(th) 1.0 to 2.5V, Vds 20V min,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
Changed lines of the file:
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@@
 <attribute name="SPEC" value="thick film +-1%, 1/16W, 0402"/>
 </part>
-<part name="LD5" library="ctambe" deviceset="LED" device=""/>
-<part name="Q2" library="ctambe" deviceset="NMOS" device=""/>
+<part name="LD5" library="ctambe" deviceset="LED" device="" value="green">
+<attribute name="MANF" value="Lite-On"/>
+<attribute name="MANF#" value="LTST-C191KGKT"/>
+<attribute name="SPEC" value="green indicator, 0603, Vf 2.1V max at 2mA"/>
+<attribute name="NOTE" value="Power-good indicator: VCC3V3 to LD5 to R78 680R to Q2 drain to GND. SELECTED FROM THE CIRCUIT, not recovered -- the part carried no value and no number. THE RESISTOR ALREADY CHOSE THE COLOUR: 680R off 3.3 V passes (3.3 - Vf)/680, which is 1.9 mA for a green LED or 2.1 for a red, but only 0.6 mA for a blue or white one, too dim to read. So it is a green or red part, and green is the convention for power good. 1.9 mA is low but plain on a modern high-efficiency 0603; take R78 to 330R if you want it brighter."/>
+</part>
+<part name="Q2" library="ctambe" deviceset="NMOS" device="" value="2N7002">
+<attribute name="MANF" value="onsemi"/>
+<attribute name="MANF#" value="2N7002LT1G"/>
+<attribute name="SPEC" value="N-ch MOSFET, logic level: Vgs(th) 1.0 to 2.5V, Vds 20V min, Id 100mA min, SOT-23 G/S/D on pins 1/2/3"/>
+<attribute name="NOTE" value="Switches the PGOOD indicator LD5. SELECTED FROM THE CIRCUIT, not recovered -- the part carried no value and no number. What it has to do: its gate is on PGOOD, the LTC3569's open-drain output pulled to 3V3 through R77's 100k, so Vgs is a static 3.3 V and the weak pull-up costs nothing because a gate draws no DC. That needs a LOGIC-LEVEL threshold, comfortably under 3.3 V. The drain carries the LED at 1.9 mA against the 2N7002's 115 mA, and sees 3.3 V against 60. The SOT23-3 footprint here names its pads G, S and D at pins 1, 2 and 3, which is the 2N7002 pinout exactly, so nothing in the layout moves."/>
+</part>
 <part name="GND8" library="ctambe" deviceset="GND" device=""/>
 <part name="X1" library="ctambe" deviceset="MINI-USB-" device="105017-0001" value="Molex 105017-0001 Micro-USB-B"/>
