File: zulu_a7.sch (EAGLE design)
At the start: 183 parts, among them J1 Pmod 2x6, Q1 12MHz 25ppm (FPGA + FT2232HQ), Q2 2N7002, Q3 MBT3904DW1T1, U1 XC7A35T-1CPG236C, U10 93LC46BT-I/SN, U2 FT2232HQ USB-UART/JTAG Bridge, U3 AS4C32M16SB-6TIN, U4 W25Q128JVSIQ, U8 LTC3569EUDC#TRPBF, X1 Molex 105017-0001 Micro-USB-B, X2 ZULU-CONN, X3 MICROSD_CONDM3AT-SF-PEJM5

Commit message: BTN and LD0 from their datasheets; every part now has a number
Both were in Datasheet/, and both turned out to have had their number in the
value field all along -- I had called them series names, and for these two that
was wrong.

LD0 -> VS NRD8, Victory Electronics. The datasheet's own "Part Number" column
reads VS NRD8, so it is the part, not a family. Confirmed against the drawing
this library's land was traced from.

BTN -> PTA-142. The catalogue page is IMAGE-ONLY -- twelve JPEGs, no text layer
at all -- so pdf text extraction returned nothing and I had to render it and read
the picture. It says the part number is complete as it stands: one operating
force (130 gf +-30), one stem colour, and no ordering suffix table. It is the
SMD reflow member of the family; PTA-112 and PTA-113 are through-hole and
PTA-143 is the SMD with a ground terminal. Its P.C.B. Layout -- 9.1 overall, 5.9
inner, 4.4 high, 1.6 pads -- is exactly the land in this library, which confirms
the footprint came from this page. THE PAGE NAMES NO MANUFACTURER: it is one
sheet out of a catalogue with a decorative banner and no logo, so MANF is left
empty rather than guessed. Distributors index PTA-142 directly.

READING THE LED DATASHEET TURNED UP SOMETHING ELSE. Vf for GREEN and BLUE is
3.3 V typical and 3.8 maximum at 20 mA, and the rail is 3.3 V. Red is properly
set: R81 at 182R gives about 6 mA. Green through R82 at 100R and blue through
R80 at 182R have no headroom at all at the typical Vf, so their current is
whatever the diode knee allows rather than what the resistor sets. They will
light, because Vf falls at low current, but dimly and with a wide part-to-part
spread, and red will dominate the mix. That is on LD0 as a NOTE. It is a design
question, not a sourcing one, and I have not changed anything for it.

Lines with no MANF# are down to X2 alone, which is the board's own pin field.
No board regenerate: no element value changed, only attributes.

Co-Authored-By: Claude Opus 5 <noreply@an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
Parts:
- BTN: MANF# (none) -> PTA-142; NOTE (none) -> PTA-142, from the catalogue page in Datasheet/pta142-112.pd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; SPEC (none) -> tactile switch, SMD gull-wing, 4.5 x 4.5 mm, 130 gf, DC12V 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
- LD0: MANF (none) -> Victory Electronics; MANF# (none) -> VS NRD8; NOTE (none) -> Victory Electronics VS NRD8, common anode, 1.6 x 1.6 x 0.35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; SPEC (none) -> RGB LED, common anode, 1.6 x 1.6 x 0.35 mm, 25 mA max per c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
Changed lines of the file:
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@@
 <attribute name="SPEC" value="thick film +-1%, 1/20W, 0201"/>
 </part>
-<part name="LD0" library="ctambe" deviceset="LED_RGB" device="" value="VS NRD8"/>
+<part name="LD0" library="ctambe" deviceset="LED_RGB" device="" value="VS NRD8">
+<attribute name="MANF" value="Victory Electronics"/>
+<attribute name="MANF#" value="VS NRD8"/>
+<attribute name="SPEC" value="RGB LED, common anode, 1.6 x 1.6 x 0.35 mm, 25 mA max per colour"/>
+<attribute name="NOTE" value="Victory Electronics VS NRD8, common anode, 1.6 x 1.6 x 0.35 mm. The datasheet's own Part Number column says VS NRD8, so the value was the part number all along. Land pattern already drawn from its Recommended Soldering Pad. 25 mA absolute max per colour; red 60 mW, green and blue 110 mW. WORTH A LOOK BEFORE FABRICATION: Vf is 3.3 V typ and 3.8 max for GREEN and BLUE at 20 mA, against a 3.3 V rail. Red is properly set -- R81 at 182R gives about 6 mA. Green through R82 at 100R and blue through R80 at 182R have NO HEADROOM at the typical Vf, so their current is set by where the diode knee happens to sit rather than by the resistor. They will light, because Vf falls at low current, but dimly and with a wide part-to-part spread. Red will dominate the mix. Options are a lower-Vf RGB part, or accepting it."/>
+</part>
 <part name="LD1" library="ctambe" deviceset="LED" device="" value="red">
 <attribute name="MANF" value="Lite-On"/>
@@
 <attribute name="NOTE" value="User status LED, driven straight off an FPGA pin through R84 at 330R: (3.3 - Vf)/330 is 3.9 mA green, 4.2 red, 3.6 yellow, and 1.2 mA blue or white. Any of the first three is comfortable and well inside an LVCMOS33 pin's 12 mA. RED IS A PREFERENCE, NOT A CONSTRAINT -- the circuit takes green just as happily. It is red so that the two user LEDs read differently from LD5, which is green and means power good; on a board being brought up that is worth being able to tell apart at a glance. Same LTST-C191 family and the same 0603 land as LD5, so it is one line in the catalogue, not two. Confirm the suffix before ordering."/>
 </part>
-<part name="BTN" library="ctambe" deviceset="SWITCH_TACT" device="" value="PTA-142"/>
+<part name="BTN" library="ctambe" deviceset="SWITCH_TACT" device="" value="PTA-142">
+<attribute name="MANF#" value="PTA-142"/>
+<attribute name="SPEC" value="tactile switch, SMD gull-wing, 4.5 x 4.5 mm, 130 gf, DC12V 50 mA, 50000 cycles"/>
+<attribute name="NOTE" value="PTA-142, from the catalogue page in Datasheet/pta142-112.pdf. THE PART NUMBER IS COMPLETE AS IT STANDS: the sheet lists one operating force (130 gf +-30), one stem colour (black) and no ordering suffix table, so there is nothing to append. It is the SMD reflow member of the family -- PTA-112 and PTA-113 are through-hole, PTA-143 is the SMD with a ground terminal. Rated DC12V 50 mA, 100 mOhm contact, 50000 cycles, 0.25 mm travel, 2200 per reel. The P.C.B. Layout on that page is 9.1 mm overall, 5.9 inner, 4.4 high, 1.6 pads, which is exactly the land in this library. THE PAGE DOES NOT NAME THE MANUFACTURER -- it is one sheet lifted out of a catalogue and carries no logo, so MANF is left empty rather than guessed. Distributors index PTA-142 directly."/>
+</part>
 <part name="Q1" library="ctambe" deviceset="OSC_CHIP" device="ASEM1-12MHZ" value="12MHz 25ppm (FPGA + FT2232HQ)">
 <attribute name="MANF" value="Abracon"/>

Commit message: Balance the RGB LED, and correct what I said was wrong with it
FIRST, THE RETRACTION. I said green and blue had "no headroom" and their current
was "set by the diode knee", implying they might barely light. That was wrong,
and the error was mine: I took Vf = 3.3 V typical from the datasheet's 20 mA
table and applied it at a 2 mA operating point. The datasheet's own Vf/If curve
on page 3 puts Vf near 3.0 V down there. Worked properly, the circuit as built
gives red 6.9 mA, green 1.9 and blue 1.5. All three light.

Cmod A7 ships the identical circuit -- same VS NRD8, same 182/182/100 off 3V3,
per its schematic in Datasheet/cmod_a7_sch.pdf. Zulu A7 inherited it whole.

WHAT IS ACTUALLY WRONG IS BALANCE, NOT HEADROOM. Red is an AlGaInP die at about
1.9 V with real margin on a 3.3 V rail; green and blue are 3.3 V-class dice with
almost none. So red ran at four times either of them and dominated every colour
the three are mixed into. Headroom itself cannot be fixed with resistors -- that
is the rail against the die -- but the imbalance can:

    R81 red    182 -> 330    6.9 mA -> 3.8
    R82 green  100 ->  33    1.9 mA -> 2.9
    R80 blue   182 ->  33    1.5 mA -> 2.9

Both new values are already on this board, so the BOM gains no line -- and the
182 ohm line disappears entirely, since R80 and R81 were the only two.

THE TRADE IS REAL AND WORTH STATING. A smaller resistor makes green's current
MORE sensitive in percentage terms: a part 0.15 V high in Vf keeps 77 percent of
nominal at 100R but only 61 at 33R. The absolute floor is what an eye sees,
though, and that rises -- 1.4 mA to 1.8. Nominal and worst case both improve.

LD0's note is rewritten to say this correctly rather than to warn about a
failure that was not there.

178 placed, check_board and validate 0 findings. Regenerated, because element
values changed.

Co-Authored-By: Claude Opus 5 <noreply@anthropic.com>
Parts:
- LD0: NOTE Victory Electronics VS NRD8, common anode, 1.6 x 1.6 x 0.35 mm. The datasheet's own Part Number column says VS NRD8, so the value was the part number all along. Land pattern already drawn from its Recommended Soldering Pad. 25 mA absolute max per colour; red 60 mW, green and blue 110 mW. WORTH A LOOK BEFORE FABRICATION: Vf is 3.3 V typ and 3.8 max for GREEN and BLUE at 20 mA, against a 3.3 V rail. Red is properly set -- R81 at 182R gives about 6 mA. Green through R82 at 100R and blue through R80 at 182R have NO HEADROOM at the typical Vf, so their current is set by where the diode knee happens to sit rather than by the resistor. They will light, because Vf falls at low current, but dimly and with a wide part-to-part spread. Red will dominate the mix. Options are a lower-Vf RGB part, or accepting it. -> Victory Electronics VS NRD8, common anode, 1.6 x 1.6 x 0.35 mm. The datasheet's own Part Number column reads VS NRD8, so the value was the part number all along. Land pattern already drawn from its Recommended Soldering Pad. 25 mA absolute max per colour. GREEN AND BLUE ARE 3.3 V-CLASS DICE ON A 3.3 V RAIL: their Vf is 3.3 V typical at 20 mA, but the working point here is 2 to 3 mA, where the datasheet curve puts Vf near 3.0, so they light perfectly well -- the 20 mA figure does not apply at 3 mA. What it does mean is that the series resistor never dominates their current, so brightness tracks the diode rather than the resistor and varies with part and temperature. Red, an AlGaInP die at about 1.9 V, has real headroom and is set by its resistor. R80, R81 and R82 are chosen to balance that as far as a 3.3 V rail allows; see the note on any of them.
- R80: value 182 -> 33; MANF# RC0402FR-07182RL -> RC0402FR-0733RL; NOTE (none) -> RGB LED balance. The green and blue dice are 3.3 V-class pa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
- R81: value 182 -> 330; MANF# RC0402FR-07182RL -> RC0402FR-07330RL; NOTE (none) -> RGB LED balance. The green and blue dice are 3.3 V-class pa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
- R82: value 100 -> 33; MANF# RC0402FR-07100RL -> RC0402FR-0733RL; NOTE (none) -> RGB LED balance. The green and blue dice are 3.3 V-class pa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
Changed lines of the file:
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@@
 <part name="FRAME6" library="ctambe" deviceset="DOCFIELD" device=""/>
 <part name="FRAME7" library="ctambe" deviceset="DOCFIELD" device=""/>
-<part name="R80" library="rcl" deviceset="R-US_SMALL" device="R0402" value="182">
+<part name="R80" library="rcl" deviceset="R-US_SMALL" device="R0402" value="33">
 <attribute name="MANF" value="Yageo"/>
-<attribute name="MANF#" value="RC0402FR-07182RL"/>
+<attribute name="MANF#" value="RC0402FR-0733RL"/>
 <attribute name="SPEC" value="thick film +-1%, 1/16W, 0402"/>
+<attribute name="NOTE" value="RGB LED balance. The green and blue dice are 3.3 V-class parts on a 3.3 V rail, so the resistor never dominates their current -- that is structural and no resistor value fixes it. What the values CAN do is stop red swamping the other two. As built, and as Cmod A7 ships the same LED, 182/182/100 gave red 6.9 mA against green 1.9 and blue 1.5: red about four times either. At 330/33/33 it is red 3.8, green 2.9, blue 2.9. Worst case improves too, not just nominal -- green with a part 0.15 V high in Vf goes from 1.4 mA to 1.8. Lower resistors do make the current MORE sensitive in percentage terms, 77 percent of nominal retained at 100R against 61 at 33R, but the absolute floor is what you see and it rises. Currents read off the datasheet's own Vf/If curve at the working point, not off the 20 mA table."/>
 </part>
-<part name="R81" library="rcl" deviceset="R-US_SMALL" device="R0402" value="182">
+<part name="R81" library="rcl" deviceset="R-US_SMALL" device="R0402" value="330">
 <attribute name="MANF" value="Yageo"/>
-<attribute name="MANF#" value="RC0402FR-07182RL"/>
+<attribute name="MANF#" value="RC0402FR-07330RL"/>
 <attribute name="SPEC" value="thick film +-1%, 1/16W, 0402"/>
+<attribute name="NOTE" value="RGB LED balance. The green and blue dice are 3.3 V-class parts on a 3.3 V rail, so the resistor never dominates their current -- that is structural and no resistor value fixes it. What the values CAN do is stop red swamping the other two. As built, and as Cmod A7 ships the same LED, 182/182/100 gave red 6.9 mA against green 1.9 and blue 1.5: red about four times either. At 330/33/33 it is red 3.8, green 2.9, blue 2.9. Worst case improves too, not just nominal -- green with a part 0.15 V high in Vf goes from 1.4 mA to 1.8. Lower resistors do make the current MORE sensitive in percentage terms, 77 percent of nominal retained at 100R against 61 at 33R, but the absolute floor is what you see and it rises. Currents read off the datasheet's own Vf/If curve at the working point, not off the 20 mA table."/>
 </part>
-<part name="R82" library="rcl" deviceset="R-US_SMALL" device="R0402" value="100">
+<part name="R82" library="rcl" deviceset="R-US_SMALL" device="R0402" value="33">
 <attribute name="MANF" value="Yageo"/>
-<attribute name="MANF#" value="RC0402FR-07100RL"/>
+<attribute name="MANF#" value="RC0402FR-0733RL"/>
 <attribute name="SPEC" value="thick film +-1%, 1/16W, 0402"/>
+<attribute name="NOTE" value="RGB LED balance. The green and blue dice are 3.3 V-class parts on a 3.3 V rail, so the resistor never dominates their current -- that is structural and no resistor value fixes it. What the values CAN do is stop red swamping the other two. As built, and as Cmod A7 ships the same LED, 182/182/100 gave red 6.9 mA against green 1.9 and blue 1.5: red about four times either. At 330/33/33 it is red 3.8, green 2.9, blue 2.9. Worst case improves too, not just nominal -- green with a part 0.15 V high in Vf goes from 1.4 mA to 1.8. Lower resistors do make the current MORE sensitive in percentage terms, 77 percent of nominal retained at 100R against 61 at 33R, but the absolute floor is what you see and it rises. Currents read off the datasheet's own Vf/If curve at the working point, not off the 20 mA table."/>
 </part>
 <part name="R83" library="rcl" deviceset="R-US_SMALL" device="R0402" value="330">
@@
 <attribute name="MANF#" value="VS NRD8"/>
 <attribute name="SPEC" value="RGB LED, common anode, 1.6 x 1.6 x 0.35 mm, 25 mA max per colour"/>
-<attribute name="NOTE" value="Victory Electronics VS NRD8, common anode, 1.6 x 1.6 x 0.35 mm. The datasheet's own Part Number column says VS NRD8, so the value was the part number all along. Land pattern already drawn from its Recommended Soldering Pad. 25 mA absolute max per colour; red 60 mW, green and blue 110 mW. WORTH A LOOK BEFORE FABRICATION: Vf is 3.3 V typ and 3.8 max for GREEN and BLUE at 20 mA, against a 3.3 V rail. Red is properly set -- R81 at 182R gives about 6 mA. Green through R82 at 100R and blue through R80 at 182R have NO HEADROOM at the typical Vf, so their current is set by where the diode knee happens to sit rather than by the resistor. They will light, because Vf falls at low current, but dimly and with a wide part-to-part spread. Red will dominate the mix. Options are a lower-Vf RGB part, or accepting it."/>
+<attribute name="NOTE" value="Victory Electronics VS NRD8, common anode, 1.6 x 1.6 x 0.35 mm. The datasheet's own Part Number column reads VS NRD8, so the value was the part number all along. Land pattern already drawn from its Recommended Soldering Pad. 25 mA absolute max per colour. GREEN AND BLUE ARE 3.3 V-CLASS DICE ON A 3.3 V RAIL: their Vf is 3.3 V typical at 20 mA, but the working point here is 2 to 3 mA, where the datasheet curve puts Vf near 3.0, so they light perfectly well -- the 20 mA figure does not apply at 3 mA. What it does mean is that the series resistor never dominates their current, so brightness tracks the diode rather than the resistor and varies with part and temperature. Red, an AlGaInP die at about 1.9 V, has real headroom and is set by its resistor. R80, R81 and R82 are chosen to balance that as far as a 3.3 V rail allows; see the note on any of them."/>
 </part>
 <part name="LD1" library="ctambe" deviceset="LED" device="" value="red">
