File: Claude_Fable/zulu_a7.c3s.brd (EAGLE design)
At the start: 69.8 x 25.4 mm, 183 parts, among them J1 Pmod 2x6, Q1 12MHz 25ppm (FPGA + FT2232HQ), Q2 2N7002, Q3 MBT3904DW1T1, U1 XC7A35T-1CPG236C, U10 93LC46BT-I/SN, U2 FT2232HQ USB-UART/JTAG Bridge, U3 AS4C32M16SB-6TIN, U4 W25Q128JVSIQ, U8 LTC3569EUDC#TRPBF, X1 Molex 105017-0001 Micro-USB-B

Commit message: Re-placed board on the 2+4+2 base, planned stubs, checkpoint after the pass
zulu_a7.c3.brd / c3s.brd: the core re-placement rebuilt on a 2+4+2 base
(the first attempt was cut from the 1+6+1 board and put signal traces on
the GND plane's layer, which is what crashed run c4). c3s adds the planned
escape stubs for 106 balls.

close_airwires.py: a checkpoint is written right after the strip-all pass,
before the plane pass and verification. STUB_R 3.0 so a longer planned
escape is kept whole.

bga_escape.py --exclude; bga_inward.py: an inward-lane planner for the
SDRAM balls (kept for the record; at 0.5 mm pitch a 0.30 mm via land
cannot sit beside 0.25 mm spaced escapes, so it places 7 of 39 lanes).

u3_via_in_pad.py finds U3's pads from the element wherever it stands.

Co-Authored-By: Claude Fable 5.1 <noreply@anthropic.com>
Routing:
- net CHAN24: track 0.35 -> 2.36 mm
- net CHAN17: track 0.35 -> 2.36 mm
- net CHAN6: track 3.75 -> 5.76 mm
- net JA10: track 0.35 -> 2.36 mm
- net JA4: track 0.35 -> 2.36 mm
- net SD-CMD: track 27.3 -> 29.1 mm
- net FPGA-INIT#: track 0.35 -> 2.15 mm
- net FPGA-DONE: track 0.35 -> 2.15 mm
- net D7: track 0.35 -> 2.15 mm
- net FPGA-CCLK: track 0.35 -> 2.15 mm
- net CHAN4: track 0.35 -> 2.15 mm
- net AIN15_P: track 0.35 -> 2.15 mm
- net CLK-12M-FPGA: track 13.0 -> 14.8 mm
- net CHAN9: track 43.3 -> 45.1 mm
- net CHAN11: track 20.4 -> 22.2 mm
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