File: Claude_Fable/zulu_a7.c3i.brd (EAGLE design)
At the start: 69.8 x 25.4 mm, 183 parts, among them J1 Pmod 2x6, Q1 12MHz 25ppm (FPGA + FT2232HQ), Q2 2N7002, Q3 MBT3904DW1T1, U1 XC7A35T-1CPG236C, U10 93LC46BT-I/SN, U2 FT2232HQ USB-UART/JTAG Bridge, U3 AS4C32M16SB-6TIN, U4 W25Q128JVSIQ, U8 LTC3569EUDC#TRPBF, X1 Molex 105017-0001 Micro-USB-B

Commit message: Commit other pending work found in the tree
Changes made outside this session (or in earlier ones) that were still uncommitted:
- Zulu_Altium_VS_Code/tools/generate_jlcpcb_assembly.py: command-line options for an
  assembler-neutral release (--pcb, --assembly-dir, --release-prefix, --release-name).
- Zulu_Altium_VS_Code zulu_a7_6.SchDoc: saved 2026-10-04 21:36.
- Zulu_Altrium zulu_a7.PcbDoc: an intermediate Phase II board saved 2026-10-02 05:15;
  the finished board is Zulu_Altium_VS_Code. Zulu_Altrium/plan.json added.
- Claude_Fable (EAGLE era): c0 board and c3 force file changes, c3i/c5p boards and
  net lists.
- W1150632AS3P1.pdf / P2.pdf: PCBWay order summaries (6 layers, 69.9 x 25.4 mm, qty 5).

Co-Authored-By: Claude Opus 5.5 <noreply@anthropic.com>
Routing:
- net VCC3V3: track 383.3 -> 360.0 mm
- net GND: track 362.3 -> 348.7 mm
- net VCC1V0: track 181.1 -> 168.8 mm
- net VU: track 154.8 -> 144.0 mm
- net GNDADC: track 20.6 -> 12.3 mm
- net VCCADC: track 36.0 -> 28.1 mm
- net VCC1V8: track 119.1 -> 115.4 mm
- net CHAN24: track 0.00 -> 2.36 mm, vias 0 -> 2
- net CHAN17: track 0.00 -> 2.36 mm, vias 0 -> 2
- net CHAN6: track 3.40 -> 5.76 mm, vias 0 -> 2
- net JA10: track 0.00 -> 2.36 mm, vias 0 -> 2
- net JA4: track 0.00 -> 2.36 mm, vias 0 -> 2
- net A7: track 34.9 -> 37.2 mm, vias 10 -> 11
- net A11: track 2.38 -> 4.73 mm, vias 1 -> 2
- net SD-DAT2: track 42.7 -> 44.8 mm, vias 5 -> 7
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