File: Zulu_kicad/kicad_project/zulu_a7_4.kicad_sch (KiCad schematic)
At the start: 38 parts, among them Q1 12MHz 10ppm (FPGA + FT2232HL), U10 93LC46BT-I/SN, U2 FT2232HL USB-UART/JTAG Bridge

Commit message: Show "AUTHOR: Christian Tambe" in every schematic title block
The EAGLE title block reads "AUTHOR: >AUTHOR" (>AUTHOR = Christian Tambe).
The Altium EAGLE importer left the DOCFIELD AUTHOR parameter as the
literal word "AUTHOR" and dropped the "AUTHOR:" label, and the KiCad
conversion inherited the placeholder.

- Altium (production and HDI_Optimized, 7 SchDocs each):
  tools/schematic_author.py sets the AUTHOR parameter to "Christian Tambe"
  and appends an "AUTHOR:" label at the PROJECT: column in its font, then
  updates the header Weight; every other record stays byte-identical.
  Checked in Altium (sheets 1 and 3) and with the ECO preview, which shows
  only the usual never-executed baseline.
- KiCad: tools/apply_schematic_author.py sets the AUTHOR property and adds
  an AUTHOR_LABEL property. PDF plot shows the row on all 7 pages; netlist
  identical, ERC 1,648 unchanged.
- Docs: docs/schematic_author.md, HDI notes, CONVERSION.md, README notices.
  Zulu_Altrium/ and Altium_backup/ are left as historical snapshots.

Co-Authored-By: Claude Opus 5.5 <noreply@anthropic.com>
Parts:
- FRAME4: AUTHOR AUTHOR -> Christian Tambe; AUTHOR_LABEL (none) -> AUTHOR:
Changed lines of the file:
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@@
 			)
 		)
-		(property "AUTHOR" "AUTHOR"
+		(property "AUTHOR" "Christian Tambe"
 			(at 86.868 290.068 90)
 			(show_name no)
 			(do_not_autoplace no)
+			(effects
+				(font
+					(size 1.27 1.27)
+				)
+				(justify right bottom)
+			)
+		)
+		(property "AUTHOR_LABEL" "AUTHOR:"
+			(at 67.818 290.068 90)
+			(show_name no)
+			(do_not_autoplace no)
